Commit message: 22-02-67

File: robot_description/robot_urdf/robot_urdf.urdf (robot description, URDF)
Before this commit: robot robot_armm, 3 links, 2 joints
Joints:
- joint joint1: origin xyz=0 0 0.07 rpy=0 0 0 -> xyz=0 0.3 0.14 rpy=0 0 0
- joint joint2: origin xyz=0.0 0.0 0.1 rpy=0 0 0 -> xyz=0.27 0 0.14 rpy=0 0 0
