Commit message: 22-02-67

File: robot_description/robot_urdf/robot.urdf (robot description, URDF)
Before this commit: robot robot_armm, 1 links, 0 joints
Links:
- added link link1, mass 0.104; collision mesh filename=package://robot_description/robot_urdf/robot_link1.stl scale=0.001 0.001 0.001; visual mesh filename=package://robot_description/robot_urdf/robot_link1.stl scale=0.001 0.001 0.001
- added link link2, mass 0.104; collision mesh filename=package://robot_description/robot_urdf/robot_link2.stl scale=0.001 0.001 0.001; visual mesh filename=package://robot_description/robot_urdf/robot_link2.stl scale=0.001 0.001 0.001
- link base_link: geometry collision mesh filename=package://robot_description/robot_urdf/robot_base.stl scale=0.001 0.001 0.001; visual mesh filename=package://robot_description/robot_urdf/robot_base.stl scale=0.001 0.001 0.001
Joints:
- added joint joint1: type prismatic, parent base_link, child link1, origin xyz=0 0 0.07 rpy=0 0 0, axis 1 0 0, limit lower=-0.15 upper=0.15 effort=100 velocity=1
- added joint joint2: type prismatic, parent base_link, child link2, origin xyz=0.0 0.0 0.1 rpy=0 0 0, axis 0 1 0, limit lower=-0.15 upper=0.15 effort=100 velocity=1
